File: board_pico2knob/pico2-knob.kicad_sch (KiCad schematic)
At the start: 30 parts, among them J2 LiPo_JST_PH, J3 ER-CON20HT-1, Q1 DMG3415U, SW1 SW_Push, SW2 SW_Push, SW3 SW_Push, U1 nice!nano_v2, U2 MC34063AD

Commit message: pre-U2 flip
Connections:
- net GND is gone; now on net +12V: C1.2, C2.2, C3.2, C4.1, C5.2, C6.2, DS1.20 (GND), DS1.4 (IM1), DS1.5 (IM2), J2.2 (Pin_2), J3.20 (Pin_20), J3.4 (Pin_4), J3.5 (Pin_5), R1.2, R4.2, RE1.C, RE1.S2, SW1.2, SW2.2, SW3.2, TP1.1, U1.14 (GND), U1.28 (GND), U1.3 (GND), U1.4 (GND), U2.2 (SwE), U2.4 (GND)
Other:
- moved on the sheet: C1, C3, C6, D1, L1, Q1, R3, R4, R5, R7, R8, U2

Commit message: passing erc/drc
Connections:
- net +12V: no longer C1.2, C2.2, C3.2, C4.1, C5.2, C6.2, DS1.20 (GND), DS1.4 (IM1), DS1.5 (IM2), J2.2 (Pin_2), J3.20 (Pin_20), J3.4 (Pin_4), J3.5 (Pin_5), R1.2, R4.2, RE1.C, RE1.S2, SW1.2, SW2.2, SW3.2, TP1.1, U1.14 (GND), U1.28 (GND), U1.3 (GND), U1.4 (GND), U2.2 (SwE), U2.4 (GND)
- new net GND: C1.2, C2.2, C3.2, C4.1, C5.2, C6.2, DS1.20 (GND), DS1.4 (IM1), DS1.5 (IM2), J2.2 (Pin_2), J3.20 (Pin_20), J3.4 (Pin_4), J3.5 (Pin_5), R1.2, R4.2, RE1.C, RE1.S2, SW1.2, SW2.2, SW3.2, TP1.1, U1.14 (GND), U1.28 (GND), U1.3 (GND), U1.4 (GND), U2.2 (SwE), U2.4 (GND)
- no-connect marks 13 -> 19
